Commit message: updated obstacles and waypointpublisher

File: src/vipnav/description/thermal_sensor.xacro (robot description, xacro)
@@ -2,15 +2,24 @@
 <robot xmlns:xacro="http://www.ros.org/wiki/xacro">
     <joint name="thermal_camera_joint" type="fixed">
-        <parent link="chassis"/>
-        <child link="thermal_camera_link"/>
-        <origin xyz="0.15 0 0.15" rpy="0 0 0"/>
+        <parent link="chassis"/> <child link="thermal_camera_link"/>
+        <origin xyz="0.15 0 0.2" rpy="0 0 0"/>
     </joint>
     <link name="thermal_camera_link">
         <visual>
             <geometry>
-                <box size="0.02 0.04 0.02"/>
+                <box size="0.02 0.05 0.03"/>
             </geometry>
             <material name="black"/>
         </visual>
+        <collision>
+            <geometry>
+                <box size="0.02 0.05 0.03"/>
+            </geometry>
+        </collision>
+        <inertial>
+            <mass value="0.1"/>
+            <origin xyz="0 0 0" rpy="0 0 0"/>
+            <inertia ixx="0.0001" ixy="0" ixz="0" iyy="0.0001" iyz="0" izz="0.0001"/>
+        </inertial>
     </link>
     <gazebo reference="thermal_camera_link">
@@ -24,14 +33,11 @@
                 <clip>
                     <near>0.1</near>
-                    <far>100</far>
+                    <far>100.0</far>
                 </clip>
             </camera>
             <always_on>1</always_on>
-            <update_rate>10</update_rate>
+            <update_rate>10.0</update_rate>
             <visualize>true</visualize>
             <topic>/thermal_camera/image_raw</topic>
-            <plugin filename="gz-sim-thermal-sensor-system" name="gz::sim::systems::ThermalSensor">
-                <min_temp>273.15</min_temp> <max_temp>500.0</max_temp>  <resolution>0.1</resolution>
-            </plugin>
         </sensor>
     </gazebo>
